File: CNCPlotter.sch (EAGLE design)
At the start: 127 parts, among them IC1 HEF4050B, IC2 MC34063, IC3 LD111733, IC4 74HC4094, IC5 ATmega32U4, IC6 DRV8811, IC7 DRV8811, J1 Servo, J10 Touchscreen, J11 Touchscreen, J12 X Motor, J13 MS1, J14 MS0, J15 Y Motor, J16 MS1, J17 MS0, J2 Z Drive, J3 ISP, J4 UART, J5 12V Supply, J6 MicroSD Card, J7 HWB, J8 USB, J9 Home Switches, Q1 16MHz

Commit message: Minor updates for v1.0 production
Parts:
- removed S1: RESET, freetronics-master-v1:TAC_SWITCH_2PIN
- J1: value Servo -> SERVO
- J12: value X Motor -> X-MOTOR
- J15: value Y Motor -> Y-MOTOR
- J2: value Z Drive -> Z-DRIVE
- J5: device SparkFun:POWER_JACKSLT -> freetronics-master-v1.1:POWER_JACKPTH
- J8: value USB -> USB-6PSMT; device freetronics-luke:USB-FT -> freetronics-jon:USB-6PSMT
Connections:
- net !RESET: no longer S1.S
- net GND: now also J5.GNDBREAK, J8.FIX1, J8.FIX2, J8.PIN1, J8.PIN2, J8.TAB1, J8.TAB2; no longer J8.SH$1, S1.P
Other:
- moved on the sheet: C1, C10, C11, C12, C13, C14, C15, C16, C17, C18, C19, C2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
